File: kicad/praktikumas/praktikumas.kicad_pcb (KiCad board)
At the start: 2 copper layers, 39.1 x 37.1 mm, 19 parts, among them J1 sp, J2 Conn_01x01_Socket, J3 sp, Q1 2n3904, Q2 2n3904, U2 LM386

Commit message: 8
Connections:
- U2 pad 2: Net-(RV1-Pad2) -> GND
- U2 pad 3: GND -> Net-(RV1-Pad2)
Routing:
- net GND: track 75.9 -> 79.4 mm
- net Net-(RV1-Pad2): track 18.7 -> 17.2 mm
Changed lines of the file:
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@@
       (net 9 "Net-(C6-Pad2)") (pintype "bidirectional") (solder_mask_margin 0.102))
     (pad "2" thru_hole circle (at -1.27 3.81) (size 1.7272 1.7272) (drill 0.8128) (layers "*.Cu" "*.Mask")
+      (net 5 "GND") (pintype "input") (solder_mask_margin 0.102))
+    (pad "3" thru_hole circle (at 1.27 3.81) (size 1.7272 1.7272) (drill 0.8128) (layers "*.Cu" "*.Mask")
       (net 13 "Net-(RV1-Pad2)") (pintype "input") (solder_mask_margin 0.102))
-    (pad "3" thru_hole circle (at 1.27 3.81) (size 1.7272 1.7272) (drill 0.8128) (layers "*.Cu" "*.Mask")
-      (net 5 "GND") (pintype "input") (solder_mask_margin 0.102))
     (pad "4" thru_hole circle (at 3.81 3.81) (size 1.7272 1.7272) (drill 0.8128) (layers "*.Cu" "*.Mask")
       (net 5 "GND") (pintype "power_in") (solder_mask_margin 0.102))
@@
   (segment (start 165.295 108.907) (end 161.29 104.902) (width 0.25) (layer "B.Cu") (net 5))
   (segment (start 165.52 108.907) (end 169.966 108.907) (width 0.25) (layer "B.Cu") (net 5))
+  (segment (start 156.6066 116.6784) (end 159.3094 116.6784) (width 0.25) (layer "B.Cu") (net 5))
   (segment (start 142.718 99.212677) (end 140.218 101.712677) (width 0.25) (layer "B.Cu") (net 5))
   (segment (start 143.704323 99.212677) (end 142.718 99.212677) (width 0.25) (layer "B.Cu") (net 5))
+  (segment (start 155.418 117.867) (end 156.6066 116.6784) (width 0.25) (layer "B.Cu") (net 5))
   (segment (start 162.998 117.867) (end 165.578 115.287) (width 0.25) (layer "B.Cu") (net 5))
+  (segment (start 159.3094 116.6784) (end 160.498 117.867) (width 0.25) (layer "B.Cu") (net 5))
   (segment (start 165.704 108.723) (end 165.52 108.907) (width 0.25) (layer "B.Cu") (net 5))
   (segment (start 160.115 93.152) (end 149.765 93.152) (width 0.25) (layer "B.Cu") (net 5))
@@
   (segment (start 160.498 117.867) (end 162.998 117.867) (width 0.25) (layer "B.Cu") (net 5))
   (segment (start 169.966 108.907) (end 170.15 108.723) (width 0.25) (layer "B.Cu") (net 5))
-  (segment (start 157.958 117.867) (end 160.498 117.867) (width 0.25) (layer "B.Cu") (net 5))
   (segment (start 161.29 104.902) (end 161.29 94.327) (width 0.25) (layer "B.Cu") (net 5))
   (segment (start 165.578 115.287) (end 169.174 115.287) (width 0.25) (layer "B.Cu") (net 5))
@@
   (segment (start 169.896 91.705) (end 166.452 91.705) (width 0.25) (layer "F.Cu") (net 12))
   (segment (start 166.452 91.705) (end 163.83 94.327) (width 0.25) (layer "F.Cu") (net 12))
-  (segment (start 156.873 116.412) (end 170.589 116.412) (width 0.25) (layer "F.Cu") (net 13))
-  (segment (start 155.418 117.867) (end 156.873 116.412) (width 0.25) (layer "F.Cu") (net 13))
-  (segment (start 170.589 116.412) (end 172.69 114.311) (width 0.25) (layer "F.Cu") (net 13))
+  (segment (start 167.9454 119.0556) (end 172.69 114.311) (width 0.25) (layer "F.Cu") (net 13))
+  (segment (start 159.1466 119.0556) (end 167.9454 119.0556) (width 0.25) (layer "F.Cu") (net 13))
+  (segment (start 157.958 117.867) (end 159.1466 119.0556) (width 0.25) (layer "F.Cu") (net 13))
 )

Commit message: 9
Parts:
- C1: footprint Capacitor_THT:CP_Axial_L11.0mm_D8.0mm_P15.00mm_Horizontal -> Capacitor_THT:CP_Radial_D6.3mm_P2.50mm
- moved R1 77.9 mm to (181.6, 36.1), turned to -90 degrees
- moved C8 75.2 mm to (188.9, 61.5), turned to 180 degrees
- moved L1 75.0 mm to (198.9, 47.8), turned to 90 degrees
- moved Q1 70.9 mm to (190.8, 42.7)
- moved Q2 70.8 mm to (195.6, 42.7)
- moved C6 70.6 mm to (185.3, 56.1), turned to 0 degrees
- moved RV1 69.8 mm to (186.6, 45.5), turned to 90 degrees
- moved C2 67.6 mm to (185.9, 42.1)
- moved C7 67.5 mm to (195.1, 59.1)
- moved J2 66.6 mm to (189.7, 36.8), turned to 180 degrees
- moved R2 64.0 mm to (192.5, 74.9), turned to 180 degrees
- moved C1 63.2 mm to (195.1, 48.3), turned to 180 degrees
- moved C3 61.5 mm to (177.6, 49.3), turned to 0 degrees
- moved J3 55.7 mm to (178.1, 45.5)
- moved U2 55.4 mm to (188.0, 68.3), turned to 180 degrees
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Routing:
- net Net-(C8-Pad2): track 53.8 -> 23.8 mm
- net Net-(J1-Pin_1): track 7.15 -> 26.6 mm
- net +5V: track 34.5 -> 52.7 mm
- net Net-(Q1-E): track 31.7 -> 46.7 mm
- net GND: track 79.4 -> 90.7 mm
- net Net-(C6-Pad1): track 9.22 -> 20.4 mm
- net Net-(C8-Pad1): track 14.3 -> 21.0 mm
- net Net-(C6-Pad2): track 5.69 -> 10.0 mm
- net Net-(C3-Pad2): track 9.12 -> 5.61 mm
- net Net-(C5-Pad1): track 11.2 -> 12.4 mm
Other:
- board size 39.1 x 37.1 mm -> 29 x 42.7 mm
- board text added: "VCC"
- board text added: "ant"
- board text added: "input"
- board text added: "output"
- board text added: "speak"
