File: kicad/praktikumas/praktikumas.kicad_sch (KiCad schematic)
At the start: 16 parts, among them J1 Speaker, U1 LM386

Commit message: 4
Parts:
- added C8: 100n, symbol Device:C
- added C9: 2.2n, symbol Device:C
- added R3: 10k, symbol Device:R
- C5: value 100u -> 470u
- C6: value 0.1u -> 47p
- Q1, Q2: value ~ -> 2n2222
Connections:
- net +5V: now also C8.2
- net GND: now also C8.1, C9.1
- net at RV1.1: now also C9.2, R3.1; no longer C2.2
- new net: C2.2, R3.2
Other:
- moved on the sheet: AE1, RV1

Commit message: 4
Parts:
- removed C9: 2.2n, symbol Device:C
- removed R3: 10k, symbol Device:R
- added C10: 10p, symbol Device:C
- C2: value 22u -> 220n
- C6: value 47p -> 47n
- RV1: value 10k -> 100k
Connections:
- net at RV1.1: now also C2.2
- net at C1.1, C2.1, L1.1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: now also C10.1; no longer AE1.1 (A)
- new net: AE1.1 (A), C10.2
Other:
- moved on the sheet: AE1

Commit message: 6
Parts:
- removed AE1: Antenna, symbol Device:Antenna
- removed U1: LM386, symbol Amplifier_Audio:LM386
- added J1, J3: sp, Connector_PinSocket_2.54mm:PinSocket_1x02_P2.54mm_Horizontal, symbol Connector:Conn_01x02_Socket
- added J2: Conn_01x01_Socket, Connector_PinSocket_2.54mm:PinSocket_1x01_P2.54mm_Horizontal, symbol Connector:Conn_01x01_Socket
- added U2: LM386, LM386:DIP08, symbol LM386:LM386
- C1: footprint (none) -> Capacitor_THT:CP_Axial_L11.0mm_D8.0mm_P15.00mm_Horizontal
- C2: renamed from C10; footprint (none) -> Capacitor_THT:C_Disc_D5.1mm_W3.2mm_P5.00mm
- C3: renamed from C2; footprint (none) -> Capacitor_THT:C_Disc_D5.1mm_W3.2mm_P5.00mm
- C4: renamed from C8; footprint (none) -> Capacitor_THT:C_Disc_D5.1mm_W3.2mm_P5.00mm
- C5: renamed from C3; footprint (none) -> Capacitor_THT:CP_Radial_D6.3mm_P2.50mm
- C6: renamed from C4; footprint (none) -> Capacitor_THT:CP_Radial_D6.3mm_P2.50mm
- C7: renamed from C5; footprint (none) -> Capacitor_THT:CP_Radial_D10.0mm_P2.50mm
- C8: renamed from C6; footprint (none) -> Capacitor_THT:C_Disc_D5.1mm_W3.2mm_P5.00mm
- C9: renamed from C7; footprint (none) -> Capacitor_THT:CP_Radial_D8.0mm_P2.50mm
- L1: footprint (none) -> Inductor_THT:L_Axial_L5.3mm_D2.2mm_P7.62mm_Horizontal_Vishay_IM-1
- Q1, Q2: value 2n2222 -> 2n3904; footprint (none) -> Package_TO_SOT_THT:TO-92L_Inline
- R1, R2: footprint (none) -> Resistor_THT:R_Axial_DIN0207_L6.3mm_D2.5mm_P10.16mm_Horizontal
- RV1: footprint (none) -> Potentiometer_THT:Potentiometer_Bourns_3266Y_Vertical
- renumbered J1 to #J2
Connections:
- net +5V: now also J3.1 (Pin_1), U2.6
- net GND: now also J1.2 (Pin_2), J3.2 (Pin_2), U2.3, U2.4; no longer #J2.1-
- net at C8.2, C9.1: now also U2.5
- net at C9.2: now also J1.1 (Pin_1); no longer #J2.1+
- net at C2.2: now also J2.1 (Pin_1)
- net at C6.2: now also U2.1
- net at RV1.2: now also U2.2
- net at C5.1: now also U2.7
- net at C6.1: now also U2.8
Other:
- moved on the sheet: C5, C6

Commit message: 7
Connections:
- net GND: now also U2.2; no longer U2.3
- net at RV1.2: now also U2.3; no longer U2.2
Changed lines of the file:
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@@
   (junction (at 130.81 110.49) (diameter 0) (color 0 0 0 0)
   )
-  (junction (at 158.75 110.49) (diameter 0) (color 0 0 0 0)
-  )
   (junction (at 167.64 110.49) (diameter 0) (color 0 0 0 0)
   )
@@
     (stroke (width 0) (type default))
   )
-  (wire (pts (xy 158.75 110.49) (xy 165.1 110.49))
+  (wire (pts (xy 157.48 110.49) (xy 165.1 110.49))
     (stroke (width 0) (type default))
   )
@@
     (stroke (width 0) (type default))
   )
+  (wire (pts (xy 154.94 88.9) (xy 154.94 91.44))
+    (stroke (width 0) (type default))
+  )
+  (wire (pts (xy 154.94 88.9) (xy 160.02 88.9))
+    (stroke (width 0) (type default))
+  )
   (wire (pts (xy 128.27 57.15) (xy 128.27 54.61))
     (stroke (width 0) (type default))
@@
     (stroke (width 0) (type default))
   )
-  (wire (pts (xy 158.75 110.49) (xy 157.48 110.49))
+  (wire (pts (xy 157.48 83.82) (xy 157.48 110.49))
     (stroke (width 0) (type default))
   )
@@
     (stroke (width 0) (type dash) (color 255 0 255 1))
   )
-  (wire (pts (xy 154.94 91.44) (xy 154.94 83.82))
-    (stroke (width 0) (type default))
-  )
   (wire (pts (xy 193.04 59.69) (xy 193.04 57.15))
     (stroke (width 0) (type dash) (color 255 0 255 1))
@@
     (stroke (width 0) (type default))
   )
-  (wire (pts (xy 158.75 88.9) (xy 160.02 88.9))
-    (stroke (width 0) (type default))
-  )
   (wire (pts (xy 189.23 57.15) (xy 193.04 57.15))
     (stroke (width 0) (type dash) (color 255 0 255 1))
@@
     (stroke (width 0) (type default))
   )
+  (wire (pts (xy 160.02 83.82) (xy 157.48 83.82))
+    (stroke (width 0) (type default))
+  )
   (wire (pts (xy 114.3 54.61) (xy 128.27 54.61))
     (stroke (width 0) (type default))
@@
   )
   (wire (pts (xy 101.6 54.61) (xy 114.3 54.61))
-    (stroke (width 0) (type default))
-  )
-  (wire (pts (xy 154.94 83.82) (xy 160.02 83.82))
-    (stroke (width 0) (type default))
-  )
-  (wire (pts (xy 158.75 88.9) (xy 158.75 110.49))
     (stroke (width 0) (type default))
   )
@@
       (effects (font (size 1.27 1.27)) hide)
     )
-    (property "Value" "GND" (at 175.26 87.63 0)
+    (property "Value" "GND" (at 195.58 63.5 0)
       (effects (font (size 1.27 1.27)))
     )
@@
       (effects (font (size 1.27 1.27)) hide)
     )
-    (property "Value" "GND" (at 166.37 95.25 0)
+    (property "Value" "GND" (at 186.69 67.31 0)
       (effects (font (size 1.27 1.27)))
     )
@@
       (effects (font (size 1.27 1.27)) hide)
     )
-    (property "Value" "GND" (at 158.75 96.52 0)
-      (effects (font (size 1.27 1.27)))
-    )
+    (property "Value" "GND" (at 179.07 68.58 0)
+      (effects (font (size 1.27 1.27)))
+    )

Commit message: 9
Parts:
- C1: footprint Capacitor_THT:CP_Axial_L11.0mm_D8.0mm_P15.00mm_Horizontal -> Capacitor_THT:CP_Radial_D6.3mm_P2.50mm
Changed lines of the file:
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@@
       (effects (font (size 1.27 1.27)) (justify left))
     )
-    (property "Footprint" "Capacitor_THT:CP_Axial_L11.0mm_D8.0mm_P15.00mm_Horizontal" (at 114.3 60.96 0)
+    (property "Footprint" "Capacitor_THT:CP_Radial_D6.3mm_P2.50mm" (at 114.3 60.96 0)
       (effects (font (size 1.27 1.27)) hide)
     )
